Commit message: Implementazione del giunto rotoidale sulla staffa della camera

File: ros_ws/src/turtlebot4/turtlebot4_description/urdf/sensors/camera_bracket.urdf.xacro (robot description, xacro)
@@ -6,8 +6,16 @@
   <xacro:property name="link_name" value="${name}"/>
   <xacro:property name="joint_name" value="${name}_joint"/>
-  <joint name="${joint_name}" type="fixed">
+  <!-- <joint name="${joint_name}" type="fixed">
     <parent link="${parent_link}"/>
     <child link="${link_name}"/>
     <xacro:insert_block name="origin"/>
+  </joint> -->
+  <joint name="${joint_name}" type="continuous">
+    <parent link="${parent_link}"/>
+    <child link="${link_name}"/>
+    <xacro:insert_block name="origin"/>
+    <axis xyz="0 0 1"/>
+    # attrito e smorzamento
+    <dynamics damping="0.5" friction="0.2"/>
   </joint>
   <link name="${link_name}">

File: ros_ws/src/turtlebot4/turtlebot4_description/urdf/sensors/oakd.urdf.xacro (robot description, xacro)
@@ -14,9 +14,14 @@
   <xacro:property name="base_frame" value="${name}_link"/>
   <!-- Base frame -->
-  <joint name="${name}_joint" type="continuous">
+  <!-- <joint name="${name}_joint" type="continuous">
     <parent link="${parent_link}"/>
     <child link="${base_frame}"/>
     <xacro:insert_block name="origin"/>
     <axis xyz="0 0 1"/>
+  </joint> -->
+  <joint name="${name}_joint" type="fixed">
+    <parent link="${parent_link}"/>
+    <child link="${base_frame}"/>
+    <xacro:insert_block name="origin"/>
   </joint>
   <link name="${base_frame}">

Commit message: Il Modndo dopo il run, crusha dopo pochi secondi, eventuali problemi col file xarco

File: ros_ws/src/turtlebot4/turtlebot4_description/urdf/sensors/camera_bracket.urdf.xacro (robot description, xacro)
@@ -6,9 +6,4 @@
   <xacro:property name="link_name" value="${name}"/>
   <xacro:property name="joint_name" value="${name}_joint"/>
-  <!-- <joint name="${joint_name}" type="fixed">
-    <parent link="${parent_link}"/>
-    <child link="${link_name}"/>
-    <xacro:insert_block name="origin"/>
-  </joint> -->
   <joint name="${joint_name}" type="continuous">
     <parent link="${parent_link}"/>
@@ -16,6 +11,8 @@
     <xacro:insert_block name="origin"/>
     <axis xyz="0 0 1"/>
-    # attrito e smorzamento
-    <dynamics damping="0.5" friction="0.2"/>
+    <!-- attrito e smorzamento -->
+    <dynamics damping="0.001" friction="0.001"/>
+    <!-- limiti di velocità e movimento obbligatori -->
+    <limit lower="-1.57" upper="1.57" effort="10.0" velocity="1.0"/>
   </joint>
   <link name="${link_name}">
@@ -28,10 +25,8 @@
       <mass value="${mass}"/>
       <inertia ixx="0.0000579181" ixy="0.0" ixz="0.0000090679"
-	             iyy="0.0000559785" iyz="0.0" izz="0.0000140955" />
+               iyy="0.0000559785" iyz="0.0" izz="0.0000140955" />
     </inertial>
   </link>
-  <gazebo reference="${joint_name}">
-    <preserveFixedJoint>true</preserveFixedJoint>
-  </gazebo>
+  <!-- Il blocco preserveFixedJoint è stato rimosso appositamente -->
   <gazebo reference="${link_name}">
     <xacro:material_black/>

Commit message: cosa abbiamo fatto

File: ros_ws/src/turtlebot4/turtlebot4_description/urdf/sensors/camera_bracket.urdf.xacro (robot description, xacro)
@@ -11,8 +11,6 @@
     <xacro:insert_block name="origin"/>
     <axis xyz="0 0 1"/>
-    <!-- attrito e smorzamento -->
-    <dynamics damping="0.001" friction="0.001"/>
-    <!-- limiti di velocità e movimento obbligatori -->
-    <limit lower="-1.57" upper="1.57" effort="10.0" velocity="1.0"/>
+    <dynamics damping="0.1" friction="0.1"/>
+    <limit effort="10.0" velocity="1.0"/>
   </joint>
   <link name="${link_name}">

File: ros_ws/src/turtlebot4/turtlebot4_description/urdf/standard/turtlebot4.urdf.xacro (robot description, xacro)
@@ -24,5 +24,5 @@
   <xacro:property name="tower_standoff_z_offset"       value="${14.757*cm2m}"/>
   <xacro:property name="tower_sensor_plate_z_offset"   value="${25.257*cm2m}"/>
-  <xacro:property name="rplidar_x_offset"              value="${-4*cm2m}"/>
+  <xacro:property name="rplidar_x_offset"              value="${4*cm2m}"/>
   <xacro:property name="rplidar_y_offset"              value="${0*cm2m}"/>
   <xacro:property name="rplidar_z_offset"              value="${9.8715*cm2m}"/>
@@ -74,20 +74,4 @@
             rpy="${pi} 0 0"/>
   </xacro:weight_block>
-  <!-- Turtlebot4 tower definition -->
-  <xacro:tower_standoff name="front_left_tower_standoff">
-    <origin xyz="${front_tower_standoff_x_offset} ${front_tower_standoff_y_offset} ${tower_standoff_z_offset}"/>
-  </xacro:tower_standoff>
-  <xacro:tower_standoff name="front_right_tower_standoff">
-    <origin xyz="${front_tower_standoff_x_offset} ${-front_tower_standoff_y_offset} ${tower_standoff_z_offset}"/>
-  </xacro:tower_standoff>
-  <xacro:tower_standoff name="rear_left_tower_standoff">
-    <origin xyz="${rear_tower_standoff_x_offset} ${rear_tower_standoff_y_offset} ${tower_standoff_z_offset}"/>
-  </xacro:tower_standoff>
-  <xacro:tower_standoff name="rear_right_tower_standoff">
-    <origin xyz="${rear_tower_standoff_x_offset} ${-rear_tower_standoff_y_offset} ${tower_standoff_z_offset}"/>
-  </xacro:tower_standoff>
-  <xacro:tower_sensor_plate name="tower_sensor_plate">
-    <origin xyz="0 0 ${tower_sensor_plate_z_offset}"/>
-  </xacro:tower_sensor_plate>
   <!-- Turtlebot4 sensor definitions -->
   <xacro:rplidar name="rplidar" parent_link="shell_link" gazebo="$(arg gazebo)">
