Commit message: Ritorno all commit 11 perchè negli ultimi due incontri abbiam riscontrato diversi problemi

File: ros_ws/src/turtlebot4/turtlebot4_description/urdf/sensors/camera_bracket.urdf.xacro (robot description, xacro)
@@ -6,5 +6,5 @@
   <xacro:property name="link_name" value="${name}"/>
   <xacro:property name="joint_name" value="${name}_joint"/>
-  <joint name="${joint_name}" type="continuous">
+  <joint name="${joint_name}" type="fixed">
     <parent link="${parent_link}"/>
     <child link="${link_name}"/>
