Commit message: Pulizia del ws e modifica del Dockerfile 3.5

File: ros_ws/src/turtlebot4/turtlebot4_description/urdf/sensors/oakd.urdf.xacro (robot description, xacro)
@@ -13,11 +13,4 @@
   <xacro:property name="collision_offset_z"   value="${-0.5*cm2m}" />
   <xacro:property name="base_frame" value="${name}_link"/>
-  <!-- Base frame -->
-  <!-- <joint name="${name}_joint" type="continuous">
-    <parent link="${parent_link}"/>
-    <child link="${base_frame}"/>
-    <xacro:insert_block name="origin"/>
-    <axis xyz="0 0 1"/>
-  </joint> -->
   <joint name="${name}_joint" type="fixed">
     <parent link="${parent_link}"/>

File: ros_ws/src/turtlebot4/turtlebot4_description/urdf/standard/turtlebot4.urdf.xacro (robot description, xacro)
@@ -74,4 +74,20 @@
             rpy="${pi} 0 0"/>
   </xacro:weight_block>
+  <!-- Turtlebot4 tower definition -->
+  <!-- <xacro:tower_standoff name="front_left_tower_standoff">
+    <origin xyz="${front_tower_standoff_x_offset} ${front_tower_standoff_y_offset} ${tower_standoff_z_offset}"/>
+  </xacro:tower_standoff>
+  <xacro:tower_standoff name="front_right_tower_standoff">
+    <origin xyz="${front_tower_standoff_x_offset} ${-front_tower_standoff_y_offset} ${tower_standoff_z_offset}"/>
+  </xacro:tower_standoff>
+  <xacro:tower_standoff name="rear_left_tower_standoff">
+    <origin xyz="${rear_tower_standoff_x_offset} ${rear_tower_standoff_y_offset} ${tower_standoff_z_offset}"/>
+  </xacro:tower_standoff>
+  <xacro:tower_standoff name="rear_right_tower_standoff">
+    <origin xyz="${rear_tower_standoff_x_offset} ${-rear_tower_standoff_y_offset} ${tower_standoff_z_offset}"/>
+  </xacro:tower_standoff>
+  <xacro:tower_sensor_plate name="tower_sensor_plate">
+    <origin xyz="0 0 ${tower_sensor_plate_z_offset}"/>
+  </xacro:tower_sensor_plate> -->
   <!-- Turtlebot4 sensor definitions -->
   <xacro:rplidar name="rplidar" parent_link="shell_link" gazebo="$(arg gazebo)">
