Commit message: Giunto correttamente funzionante e plug-in correttamente caricati

File: ros_ws/src/turtlebot4/turtlebot4_description/urdf/lite/turtlebot4.urdf.xacro (robot description, xacro)
@@ -35,3 +35,25 @@
     <child link="base_footprint" />
   </joint>
+<!-- il plugin per il giunto della staffa -->
+<gazebo>
+    <plugin filename="gz-sim-joint-controller-system" name="gz::sim::systems::JointController">
+      <joint_name>oakd_camera_bracket_joint</joint_name>
+      <topic>bracket_vel</topic>
+    </plugin>
+  </gazebo>
+<!-- il plugin per muovere le ruote -->
+<gazebo>
+    <plugin filename="gz-sim-diff-drive-system" name="gz::sim::systems::DiffDrive">
+      <left_joint>left_wheel_joint</left_joint>
+      <right_joint>right_wheel_joint</right_joint>
+      <wheel_separation>0.233</wheel_separation>
+      <wheel_radius>0.03575</wheel_radius>
+      <odom_publish_frequency>30</odom_publish_frequency>
+      <topic>cmd_vel</topic>
+      <odom_topic>odom</odom_topic>
+      <tf_topic>tf</tf_topic>
+      <frame_id>odom</frame_id>
+      <child_frame_id>base_footprint</child_frame_id>
+    </plugin>
+  </gazebo>
 </robot>

File: ros_ws/src/turtlebot4/turtlebot4_description/urdf/sensors/camera_bracket.urdf.xacro (robot description, xacro)
@@ -6,11 +6,11 @@
   <xacro:property name="link_name" value="${name}"/>
   <xacro:property name="joint_name" value="${name}_joint"/>
-  <joint name="${joint_name}" type="fixed">
+  <joint name="${joint_name}" type="continuous">
     <parent link="${parent_link}"/>
     <child link="${link_name}"/>
     <xacro:insert_block name="origin"/>
     <axis xyz="0 0 1"/>
+    <limit effort="10.0" velocity="1.0"/>
     <dynamics damping="0.1" friction="0.1"/>
-    <limit effort="10.0" velocity="1.0"/>
   </joint>
   <link name="${link_name}">

Commit message: sistema con flotta e global manager implementati

File: ros_ws/src/turtlebot4/turtlebot4_description/urdf/lite/turtlebot4.urdf.xacro (robot description, xacro)
@@ -1,4 +1,10 @@
 <?xml version="1.0" ?>
 <robot name="turtlebot4" xmlns:xacro="http://ros.org/wiki/xacro">
+  <!-- ========================================== -->
+  <!-- 1. GESTIONE DEL NAMESPACE -->
+  <!-- ========================================== -->
+  <xacro:arg name="namespace" default=""/>
+  <xacro:property name="ns" value="$(arg namespace)"/>
+  <xacro:property name="tf_prefix" value="${ns + '/' if ns != '' else ''}"/>
   <!-- Base create3 model -->
   <xacro:include filename="$(find irobot_create_description)/urdf/create3.urdf.xacro" />
@@ -17,5 +23,5 @@
   <xacro:property name="oakd_lite_z_offset"             value="${9.25385*cm2m}"/>
   <!-- Turtlebot4 sensor definitions -->
-  <xacro:rplidar name="rplidar" parent_link="base_link" gazebo="$(arg gazebo)">
+  <xacro:rplidar name="rplidar" parent_link="base_link" tf_prefix="${tf_prefix}" gazebo="$(arg gazebo)">
     <origin xyz="${rplidar_x_offset} ${rplidar_y_offset} ${rplidar_z_offset + base_link_z_offset}"
             rpy="0 0 ${pi/2}"/>
@@ -24,5 +30,5 @@
     <origin xyz="${camera_mount_x_offset} ${camera_mount_y_offset} ${camera_mount_z_offset + base_link_z_offset}"/>
   </xacro:camera_bracket>
-  <xacro:oakd model="lite" parent_link="oakd_camera_bracket">
+  <xacro:oakd model="lite" parent_link="oakd_camera_bracket" tf_prefix="${tf_prefix}">
     <origin xyz="${oakd_lite_x_offset} ${oakd_lite_y_offset} ${oakd_lite_z_offset}"/>
   </xacro:oakd>
@@ -30,24 +36,26 @@
   <link name="base_footprint" />
   <joint name="base_footprint_joint" type="fixed">
-    <!-- Create3's base_link is already on the ground -->
     <origin xyz="0 0 0" rpy="0 0 0" />
     <parent link="base_link" />
     <child link="base_footprint" />
   </joint>
-  <!-- il plugin per CONTROLLARE il giunto della staffa (Input) -->
+  <!-- ========================================== -->
+  <!-- 2. I PLUGIN GAZEBO -->
+  <!-- ========================================== -->
+  <!-- Plugin per CONTROLLARE la staffa -->
   <gazebo>
     <plugin filename="gz-sim-joint-controller-system" name="gz::sim::systems::JointController">
       <joint_name>oakd_camera_bracket_joint</joint_name>
-      <topic>bracket_vel</topic>
+      <topic>${ns}/bracket_vel</topic>
     </plugin>
   </gazebo>
-  <!-- NUOVO PLUGIN: per LEGGERE lo stato del giunto della staffa (Feedback) -->
+  <!-- Plugin per LEGGERE la staffa -->
   <gazebo>
     <plugin filename="gz-sim-joint-state-publisher-system" name="gz::sim::systems::JointStatePublisher">
-      <topic>bracket_joint_state</topic>
+      <topic>${ns}/bracket_joint_state</topic>
       <joint_name>oakd_camera_bracket_joint</joint_name>
     </plugin>
   </gazebo>
-  <!-- il plugin per muovere le ruote -->
+  <!-- Plugin per muovere le ruote -->
   <gazebo>
     <plugin filename="gz-sim-diff-drive-system" name="gz::sim::systems::DiffDrive">
@@ -57,10 +65,15 @@
       <wheel_radius>0.03575</wheel_radius>
       <odom_publish_frequency>30</odom_publish_frequency>
-      <topic>cmd_vel</topic>
-      <odom_topic>odom</odom_topic>
-      <tf_topic>tf</tf_topic>
-      <frame_id>odom</frame_id>
-      <!-- QUESTA E' LA RIGA CHE GEM MI HA FATTO MODIFICARE NEL PLUGIN -->
-      <child_frame_id>base_link</child_frame_id>
+      <!-- Attivazione TF Nativo -->
+      <publish_odom>true</publish_odom>
+      <publish_odom_tf>true</publish_odom_tf>
+      <publish_wheel_tf>true</publish_wheel_tf>
+      <!-- I Topic usano il namespace normale -->
+      <topic>${ns}/cmd_vel</topic>
+      <odom_topic>${ns}/odom</odom_topic>
+      <tf_topic>/tf</tf_topic>
+      <!-- Frame ID per il TF con prefisso -->
+      <frame_id>${tf_prefix}odom</frame_id>
+      <child_frame_id>${tf_prefix}base_link</child_frame_id>
     </plugin>
   </gazebo>

File: ros_ws/src/turtlebot4/turtlebot4_description/urdf/sensors/oakd.urdf.xacro (robot description, xacro)
@@ -1,5 +1,5 @@
 <?xml version="1.0"?>
 <robot xmlns:xacro="http://ros.org/wiki/xacro">
-<xacro:macro name="oakd" params="name:=oakd parent_link *origin model:=pro">
+<xacro:macro name="oakd" params="name:=oakd parent_link tf_prefix:='' *origin model:=pro">
   <xacro:include filename="$(find irobot_create_description)/urdf/common_properties.urdf.xacro"/>
   <xacro:property name="mass"       value="0.061"/>
@@ -33,5 +33,5 @@
       <mass value="${mass}"/>
       <inertia ixx="0.00000202475" ixy="0.0" ixz="0.0"
-	             iyy="0.00001527320" iyz="0.0" izz="0.00001605536" />
+               iyy="0.00001527320" iyz="0.0" izz="0.00001605536" />
     </inertial>
   </link>
@@ -99,4 +99,6 @@
   <gazebo reference="${name}_rgb_camera_frame">
     <sensor name="rgbd_camera" type="rgbd_camera">
+      <!-- ECCO L'UNICO POSTO DOVE SERVE IL PREFISSO -->
+      <gz_frame_id>${tf_prefix}${name}_rgb_camera_frame</gz_frame_id>
       <camera>
         <horizontal_fov>1.25</horizontal_fov>
@@ -109,5 +111,6 @@
           <far>100</far>
         </clip>
-        <optical_frame_id>${name}_rgb_camera_optical_frame</optical_frame_id>
+        <!-- E QUI PER L'OPTICAL FRAME -->
+        <optical_frame_id>${tf_prefix}${name}_rgb_camera_optical_frame</optical_frame_id>
       </camera>
       <always_on>1</always_on>
@@ -117,7 +120,4 @@
     <xacro:material_darkgray/>
   </gazebo>
-  <!-- <gazebo reference="${name}_joint">
-    <preserveFixedJoint>true</preserveFixedJoint>
-  </gazebo> -->
   <gazebo reference="${name}_rgb_camera_joint">
     <preserveFixedJoint>true</preserveFixedJoint>

File: ros_ws/src/turtlebot4/turtlebot4_description/urdf/sensors/rplidar.urdf.xacro (robot description, xacro)
@@ -1,5 +1,5 @@
 <?xml version="1.0"?>
 <robot xmlns:xacro="http://ros.org/wiki/xacro">
-<xacro:macro name="rplidar" params="name parent_link gazebo *origin">
+<xacro:macro name="rplidar" params="name parent_link tf_prefix:='' gazebo *origin">
   <xacro:include filename="$(find irobot_create_description)/urdf/common_properties.urdf.xacro"/>
   <xacro:property name="mass"       value="0.17"/>
@@ -29,7 +29,7 @@
     <xacro:inertial_cuboid mass="0.17" x="${length_x}" y="${length_y}" z="${length_z}"/>
   </link>
-<!-- QUESTO E' IL BLOCCO CHE HO SOSTITUITO PER RISOLVERE IL PROBLEMA DEL LIDAR -->
 <gazebo reference="${name}_link">
     <sensor type="gpu_lidar" name="${name}">
+      <gz_frame_id>${tf_prefix}${name}_link</gz_frame_id>
       <always_on>true</always_on>
       <visualize>true</visualize>
@@ -52,5 +52,5 @@
     </sensor>
     <xacro:material_darkgray/>
-  </gazebo>
+</gazebo>
   <gazebo reference="${name}_joint">
     <preserveFixedJoint>true</preserveFixedJoint>
